Commit message: auto commit: 2025-08-29 03:02:01

File: limo_ros2/limo_description/urdf/limo_four_diff.xacro (robot description, xacro)
@@ -12,5 +12,5 @@
     <xacro:property name="track" value="0.13"/>
     <xacro:property name="wheel_vertical_offset" value="-0.10" />
-    <xacro:property name="base_mass" value="2.1557"/>
+    <xacro:property name="base_mass" value="8.0"/>
     <xacro:property name="wheel_length" value="0.045" />
     <xacro:property name="wheel_radius" value="0.045" />
@@ -39,5 +39,5 @@
     <link name="inertial_link">
         <inertial>
-            <origin xyz="0.0 0.0 0.0" />
+            <origin xyz="0.0 0.0 -0.06" />
             <mass value="${base_mass}" />
             <inertia ixx="0.24" ixy="0" ixz="0"
@@ -154,9 +154,9 @@
       <always_on>true</always_on>
       <visualize>true</visualize>
-      <update_rate>10</update_rate>
+      <update_rate>20</update_rate>
       <ray>
         <scan>
           <horizontal>
-            <samples>120</samples>
+            <samples>720</samples>
             <resolution>1.000000</resolution>
             <min_angle>-3.14159</min_angle>
@@ -167,5 +167,5 @@
           <min>0.3</min>
           <max>15.0</max>
-          <resolution>0.015</resolution>
+          <resolution>0.005</resolution>
         </range>
         <noise>

Commit message: auto commit: 2025-08-30 04:28:58

File: limo_ros2/limo_description/urdf/limo_four_diff.xacro (robot description, xacro)
@@ -1,18 +1,15 @@
 <?xml version="1.0"?>
 <robot name="limo_four_diff" xmlns:xacro="http://ros.org/wiki/xacro">
-    <xacro:include filename="$(find limo_description)/urdf/limo_xacro.xacro" />
-    <!-- <xacro:include filename="$(find limo_description)/urdf/limo_four_diff_2.gazebo" /> -->
-    <!-- Variables -->
-    <xacro:property name="M_PI" value="3.14159"/>
-    <!-- Vehicle Geometries -->
-    <xacro:property name="base_x_size" value="0.13" />
-    <xacro:property name="base_y_size" value="0.12" />
-    <xacro:property name="base_z_size" value="0.1" />
-    <xacro:property name="wheelbase" value="0.2"/>
-    <xacro:property name="track" value="0.13"/>
-    <xacro:property name="wheel_vertical_offset" value="-0.10" />
-    <xacro:property name="base_mass" value="8.0"/>
-    <xacro:property name="wheel_length" value="0.045" />
-    <xacro:property name="wheel_radius" value="0.045" />
+  <xacro:include filename="$(find limo_description)/urdf/limo_xacro.xacro" />
+  <!-- Vars -->
+  <xacro:property name="M_PI" value="3.14159"/>
+  <xacro:property name="base_x_size" value="0.13" />
+  <xacro:property name="base_y_size" value="0.12" />
+  <xacro:property name="base_z_size" value="0.10" />
+  <xacro:property name="wheelbase" value="0.2"/>
+  <xacro:property name="track" value="0.13"/>
+  <xacro:property name="wheel_vertical_offset" value="-0.12" />
+  <xacro:property name="wheel_length" value="0.045" />
+  <xacro:property name="wheel_radius" value="0.045" />
   <link name="base_footprint"/>
   <joint name="base_joint" type="fixed">
@@ -21,134 +18,109 @@
     <origin xyz="0.0 0.0 0.15" rpy="0 0 0"/>
   </joint>
-    <!-- Base link -->
-    <link name="base_link">
-        <visual>
-            <origin xyz="0 0 -0.15" rpy="0 0 1.57" />
-            <geometry>
-                <mesh filename="file://$(find limo_description)/meshes/limo_base.dae" scale="1 1 1"/>
-            </geometry>
-        </visual>
-        <collision>
-            <!--origin xyz="0 0 -0.15" rpy="0 0 1.57" /-->
-            <origin xyz="0 0 0" rpy="0 0 0" />
-          <geometry>
-              <box size="${base_x_size} ${base_y_size} ${base_z_size}"/>
-          </geometry>
-        </collision>
-    </link>
-    <link name="inertial_link">
-        <inertial>
-            <origin xyz="0.0 0.0 -0.06" />
-            <mass value="${base_mass}" />
-            <inertia ixx="0.24" ixy="0" ixz="0"
-                     iyy="0.96" iyz="0"
-                     izz="0.96" />
-        </inertial>
-    </link>
-    <joint name="inertial_joint" type="fixed">
-        <origin xyz="0 0 0" rpy="0 0 0" />
-        <parent link="base_link" />
-        <child link="inertial_link" />
-    </joint>
-    <xacro:limo_laser parent_prefix="base_link" frame_prefix="laser">
-        <origin xyz="0.103 0 -0.034" rpy="0 0 0"/>
-    </xacro:limo_laser>
-    <xacro:limo_depth_camera parent_prefix="base_link" frame_prefix="depth_camera">
-        <origin xyz="0.084 0 0.3" rpy="0 0 0"/>
-    </xacro:limo_depth_camera>
-    <xacro:limo_imu parent_prefix="base_link" frame_prefix="imu">
-        <origin xyz="0.0 0 -0.1" rpy="0 0 0"/>
-    </xacro:limo_imu>
-    <xacro:limo_wheel parent_prefix="base_link" wheel_prefix="front_left" reflect="1">
-        <origin xyz="${wheelbase/2} ${track/2} ${wheel_vertical_offset}" rpy="0 0  0" />
-    </xacro:limo_wheel>
-    <xacro:limo_wheel parent_prefix="base_link" wheel_prefix="front_right" reflect="-1">
-        <origin xyz="${wheelbase/2} ${-track/2} ${wheel_vertical_offset}" rpy="${M_PI} 0 0" />
-    </xacro:limo_wheel>
-    <xacro:limo_wheel parent_prefix="base_link" wheel_prefix="rear_left" reflect="1">
-        <origin xyz="${-wheelbase/2} ${track/2} ${wheel_vertical_offset}" rpy="0 0 0" />
-    </xacro:limo_wheel>
-    <xacro:limo_wheel parent_prefix="base_link" wheel_prefix="rear_right" reflect="-1">
-        <origin xyz="${-wheelbase/2} ${-track/2} ${wheel_vertical_offset}" rpy="${M_PI} 0 0" />
-    </xacro:limo_wheel>
-    <gazebo reference="imu_link">
+  <!-- Base -->
+  <link name="base_link">
+    <visual>
+      <origin xyz="0 0 -0.15" rpy="0 0 1.57" />
+      <geometry>
+        <mesh filename="file://$(find limo_description)/meshes/limo_base.dae" scale="1 1 1"/>
+      </geometry>
+    </visual>
+    <collision>
+      <origin xyz="0 0 0" rpy="0 0 0" />
+      <geometry>
+        <box size="${base_x_size} ${base_y_size} ${base_z_size}"/>
+      </geometry>
+    </collision>
+  </link>
+  <!-- 분산 질량 블록 (총합 10kg) -->
+  <link name="mass_fl">
+    <inertial>
+      <origin xyz="0.08 0.06 -0.10"/>
+      <mass value="2.5"/>
+      <inertia ixx="0.005" iyy="0.005" izz="0.005"/>
+    </inertial>
+  </link>
+  <joint name="joint_mass_fl" type="fixed">
+    <parent link="base_link"/>
+    <child link="mass_fl"/>
+  </joint>
+  <link name="mass_fr">
+    <inertial>
+      <origin xyz="0.08 -0.06 -0.10"/>
+      <mass value="2.5"/>
+      <inertia ixx="0.005" iyy="0.005" izz="0.005"/>
+    </inertial>
+  </link>
+  <joint name="joint_mass_fr" type="fixed">
+    <parent link="base_link"/>
+    <child link="mass_fr"/>
+  </joint>
+  <link name="mass_rl">
+    <inertial>
+      <origin xyz="-0.08 0.06 -0.10"/>
+      <mass value="2.5"/>
+      <inertia ixx="0.005" iyy="0.005" izz="0.005"/>
+    </inertial>
+  </link>
+  <joint name="joint_mass_rl" type="fixed">
+    <parent link="base_link"/>
+    <child link="mass_rl"/>
+  </joint>
+  <link name="mass_rr">
+    <inertial>
+      <origin xyz="-0.08 -0.06 -0.10"/>
+      <mass value="2.5"/>
+      <inertia ixx="0.005" iyy="0.005" izz="0.005"/>
+    </inertial>
+  </link>
+  <joint name="joint_mass_rr" type="fixed">
+    <parent link="base_link"/>
+    <child link="mass_rr"/>
+  </joint>
+  <!-- Sensors -->
+  <xacro:limo_laser parent_prefix="base_link" frame_prefix="laser">
+    <origin xyz="0.103 0 -0.034" rpy="0 0 0"/>
+  </xacro:limo_laser>
+  <xacro:limo_depth_camera parent_prefix="base_link" frame_prefix="depth_camera">
+    <origin xyz="0.084 0 0.3" rpy="0 0 0"/>
+  </xacro:limo_depth_camera>
+  <xacro:limo_imu parent_prefix="base_link" frame_prefix="imu">
+    <origin xyz="0.0 0 -0.1" rpy="0 0 0"/>
+  </xacro:limo_imu>
+  <!-- Wheels -->
+  <xacro:limo_wheel parent_prefix="base_link" wheel_prefix="front_left"  reflect="1">
+    <origin xyz="${wheelbase/2} ${track/2} ${wheel_vertical_offset}" rpy="0 0 0" />
+  </xacro:limo_wheel>
+  <xacro:limo_wheel parent_prefix="base_link" wheel_prefix="front_right" reflect="-1">
+    <origin xyz="${wheelbase/2} ${-track/2} ${wheel_vertical_offset}" rpy="${M_PI} 0 0" />
+  </xacro:limo_wheel>
+  <xacro:limo_wheel parent_prefix="base_link" wheel_prefix="rear_left"   reflect="1">
+    <origin xyz="${-wheelbase/2} ${track/2} ${wheel_vertical_offset}" rpy="0 0 0" />
+  </xacro:limo_wheel>
+  <xacro:limo_wheel parent_prefix="base_link" wheel_prefix="rear_right"  reflect="-1">
+    <origin xyz="${-wheelbase/2} ${-track/2} ${wheel_vertical_offset}" rpy="${M_PI} 0 0" />
+  </xacro:limo_wheel>
+  <!-- Gazebo: IMU -->
+  <gazebo reference="imu_link">
     <gravity>true</gravity>
     <sensor name="twr_imu" type="imu">
       <always_on>true</always_on>
+      <visualize>true</visualize>
       <update_rate>100</update_rate>
-      <visualize>true</visualize>
       <imu>
         <orientation>
-          <x>
-            <noise type="gaussian">
-              <mean>0.0</mean>
-              <stddev>2e-3</stddev>
-            </noise>
-          </x>
-          <y>
-            <noise type="gaussian">
-              <mean>0.0</mean>
-              <stddev>2e-3</stddev>
-            </noise>
-          </y>
-          <z>
-            <noise type="gaussian">
-              <mean>0.0</mean>
-              <stddev>2e-3</stddev>
-            </noise>
-          </z>
+          <x><noise type="gaussian"><mean>0.0</mean><stddev>2e-3</stddev></noise></x>
+          <y><noise type="gaussian"><mean>0.0</mean><stddev>2e-3</stddev></noise></y>
+          <z><noise type="gaussian"><mean>0.0</mean><stddev>2e-3</stddev></noise></z>
         </orientation>
-        <angular_velocity>
-          <x>
-            <noise type="gaussian">
-              <mean>0.0</mean>
-              <stddev>2e-4</stddev>
-            </noise>
-          </x>
-          <y>
-            <noise type="gaussian">
-              <mean>0.0</mean>
-              <stddev>2e-4</stddev>
-            </noise>
-          </y>
-          <z>
-            <noise type="gaussian">
-              <mean>0.0</mean>
-              <stddev>2e-4</stddev>
-            </noise>
-          </z>
-        </angular_velocity>
-        <linear_acceleration>
-          <x>
-            <noise type="gaussian">
-              <mean>0.0</mean>
-              <stddev>1.7e-2</stddev>
-            </noise>
-          </x>
-          <y>
-            <noise type="gaussian">
-              <mean>0.0</mean>
-              <stddev>1.7e-2</stddev>
-            </noise>
-          </y>
-          <z>
-            <noise type="gaussian">
-              <mean>0.0</mean>
-              <stddev>1.7e-2</stddev>
-            </noise>
-          </z>
-        </linear_acceleration>
       </imu>
-      <plugin name="two_wheeled_robot_imu" filename="libgazebo_ros_imu_sensor.so">
-        <initial_orientation_as_reference>false</initial_orientation_as_reference>
+      <plugin name="imu_plugin" filename="libgazebo_ros_imu_sensor.so">
         <frame_name>imu_link</frame_name>
-        <ros>
-          <namespace>/imu</namespace>
-          <remapping>~/out:=data</remapping>
-        </ros>
+        <ros><namespace>/imu</namespace><remapping>~/out:=data</remapping></ros>
       </plugin>
     </sensor>
-</gazebo>
-<gazebo reference="laser_link">
+  </gazebo>
+  <!-- Gazebo: Laser -->
+  <gazebo reference="laser_link">
     <sensor name="laser" type="ray">
       <always_on>true</always_on>
@@ -156,27 +128,9 @@
       <update_rate>20</update_rate>
       <ray>
-        <scan>
-          <horizontal>
-            <samples>720</samples>
-            <resolution>1.000000</resolution>
-            <min_angle>-3.14159</min_angle>
-            <max_angle>3.14159</max_angle>
-          </horizontal>
-        </scan>
-        <range>
-          <min>0.3</min>
-          <max>15.0</max>
-          <resolution>0.005</resolution>
-        </range>
-        <noise>
-          <type>gaussian</type>
-          <mean>0.0</mean>
-          <stddev>0.01</stddev>
-        </noise>
+        <scan><horizontal><samples>720</samples><resolution>1.0</resolution><min_angle>-3.14</min_angle><max_angle>3.14</max_angle></horizontal></scan>
+        <range><min>0.3</min><max>15.0</max><resolution>0.005</resolution></range>
       </ray>
       <plugin name="scan" filename="libgazebo_ros_ray_sensor.so">
-        <ros>
-          <remapping>~/out:=scan</remapping>
-        </ros>
+        <ros><remapping>~/out:=scan</remapping></ros>
         <output_type>sensor_msgs/LaserScan</output_type>
         <frame_name>laser_link</frame_name>
@@ -184,95 +138,34 @@
     </sensor>
   </gazebo>
-    <gazebo reference="front_left_wheel">
-        <mu1>100</mu1>
-        <mu2>100</mu2>
-        <kp>10000000.0</kp>
-        <kd>1.0</kd>
-        <minDepth>0.01</minDepth>
-        <fdir1>1 0 0</fdir1>
-        <maxContacts value="64"/>
-    </gazebo>
-    <gazebo reference="front_right_wheel">
-        <mu1>100</mu1>
-        <mu2>100</mu2>
-        <kp>10000000.0</kp>
-        <kd>1.0</kd>
-        <minDepth>0.01</minDepth>
-        <fdir1>1 0 0</fdir1>
-        <maxContacts value="64"/>
-    </gazebo>
-    <gazebo reference="rear_left_wheel">
-        <mu1>100</mu1>
-        <mu2>100</mu2>
-        <kp>10000000.0</kp>
-        <kd>1.0</kd>
-        <minDepth>0.01</minDepth>
-        <fdir1>1 0 0</fdir1>
-        <maxContacts value="64"/>
-    </gazebo>
-    <gazebo reference="rear_right_wheel">
-        <mu1>100</mu1>
-        <mu2>100</mu2>
-        <kp>10000000.0</kp>
-        <kd>1.0</kd>
-        <minDepth>0.01</minDepth>
-        <fdir1>1 0 0</fdir1>
-        <maxContacts value="64"/>
-    </gazebo>
-    <gazebo>
-        <plugin name="four_diff_controller" filename="libgazebo_ros_diff_drive.so">
-        <update_rate>50</update_rate>
-        <num_wheel_pairs>2</num_wheel_pairs>
-        <left_joint>front_left_wheel</left_joint>
-        <right_joint>front_right_wheel</right_joint>
-        <left_joint>rear_left_wheel</left_joint>
-        <right_joint>rear_right_wheel</right_joint>
-        <wheel_separation>0.172</wheel_separation>
-        <wheel_diameter>0.09</wheel_diameter>
-        <max_wheel_torque>20</max_wheel_torque>
-        <max_wheel_acceleration>1.0</max_wheel_acceleration>
-        <command_topic>cmd_vel</command_topic>
-        <publish_odom>true</publish_odom>
-        <publish_odom_tf>true</publish_odom_tf>
-        <publish_wheel_tf>true</publish_wheel_tf>
-        <odometry_topic>odom</odometry_topic>
-        <odometry_frame>odom</odometry_frame>
-        <robot_base_frame>base_footprint</robot_base_frame>
-        <odometry_source>1</odometry_source>
-        <ros>
-            <remapping>odom:=/odometry</remapping>
-        </ros>
-        </plugin>
-    </gazebo>
-        <!-- <gazebo reference="depth_camera_link">
-          <sensor name="sensor_camera" type="depth">
-            <pose>0.0 0.0 0.0 0.0 0.0 0.0</pose>
-            <always_on>0</always_on>
-            <update_rate>1</update_rate>
-            <camera name="limo_camera">
-              <distortion>
-                <k1>0.1</k1>
-                <k2>0.2</k2>
-                <k3>0.3</k3>
-                <p1>0.4</p1>
-                <p2>0.5</p2>
-                <center>0.5 0.5</center>
-              </distortion>
-            </camera>
-            <plugin name="gazebo_ros_depth_camera_sensor" filename="libgazebo_ros_camera.so">
-              <ros>
-                <namespace>/limo</namespace>
-                <argument>limo_camera/image_raw:=limo_camera/image</argument>
-                <argument>limo_camera/image_depth:=limo_camera/depth/camera_image_depth</argument>
-                <argument>limo_camera/camera_info:=limo_camera/camera_info_raw</argument>
-                <argument>limo_camera/camera_info_depth:=limo_camera/camera_info_depth</argument>
-                <argument>limo_camera/points:=limo_camera/camera_points</argument>
-              </ros>
-              <camera_name>depth_camera_link</camera_name>
-              <frame_name>depth_camera_link</frame_name>
-              <hack_baseline>0.07</hack_baseline>
-              <min_depth>0.001</min_depth>
-            </plugin>
-        </sensor>
-          </gazebo> -->
+  <!-- Gazebo: Base friction -->
+  <gazebo reference="base_link">
+    <mu1>2.0</mu1><mu2>1.5</mu2>
+    <slip1>0.8</slip1><slip2>0.8</slip2>
+    <kp>5e6</kp><kd>500</kd>
+    <max_vel>0.2</max_vel><min_depth>0.005</min_depth>
+  </gazebo>
+  <!-- Gazebo: Wheels -->
+  <gazebo reference="front_left_wheel"><mu1>10</mu1><mu2>10</mu2></gazebo>
+  <gazebo reference="front_right_wheel"><mu1>10</mu1><mu2>10</mu2></gazebo>
+  <gazebo reference="rear_left_wheel"><mu1>10</mu1><mu2>10</mu2></gazebo>
+  <gazebo reference="rear_right_wheel"><mu1>10</mu1><mu2>10</mu2></gazebo>
+  <!-- Gazebo: Diff drive -->
+  <gazebo>
+    <plugin name="four_diff_controller" filename="libgazebo_ros_diff_drive.so">
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