Commit message: auto commit: 2025-09-15 20:58:46

File: limo_ros2/limo_description/urdf/limo_ackerman.xacro (robot description, xacro)
@@ -1,126 +1,110 @@
 <?xml version="1.0"?>
-<robot name="limo_ackerman" xmlns:xacro="http://ros.org/wiki/xacro">
-    <xacro:arg name="robot_namespace" default="/" />
-    <xacro:include filename="$(find limo_description)/urdf/limo_xacro.xacro" />
-    <xacro:include filename="$(find limo_description)/urdf/limo_steering_hinge.xacro" />
-    <xacro:include filename="$(find limo_description)/urdf/limo_ackerman.gazebo" />
-    <!-- Variables -->
-    <xacro:property name="M_PI" value="3.14159"/>
-    <!-- Vehicle Geometries -->
-    <xacro:property name="base_x_size" value="0.13" />
-    <xacro:property name="base_y_size" value="0.12" />
-    <xacro:property name="base_z_size" value="0.10" />
-    <xacro:property name="wheelbase" value="0.2"/>
-    <xacro:property name="track" value="0.14"/>
-    <xacro:property name="wheel_vertical_offset" value="-0.100998" />
-    <xacro:property name="base_mass" value="2.1557"/>
-    <xacro:property name="wheel_length" value="0.045" />
-    <xacro:property name="wheel_radius" value="0.045" />
-    <link name="base_footprint"/>
-    <joint name="base_joint" type="fixed">
+<robot name="limo_ackerman" xmlns:xacro="http://www.ros.org/wiki/xacro">
+  <!-- Args -->
+  <xacro:arg name="robot_namespace" default="/limo"/>
+  <!-- Common macros (바퀴/힌지 링크 생성 매크로 포함) -->
+  <xacro:include filename="$(find limo_description)/urdf/limo_xacro.xacro"/>
+  <xacro:include filename="$(find limo_description)/urdf/limo_steering_hinge.xacro"/>
+  <!-- ===== Vehicle parameters (변수는 include 전에 선언되어야 함) ===== -->
+  <xacro:property name="M_PI" value="3.141592653589793"/>
+  <xacro:property name="base_x_size" value="0.13"/>
+  <xacro:property name="base_y_size" value="0.12"/>
+  <xacro:property name="base_z_size" value="0.10"/>
+  <!-- 차체 치수 -->
+  <xacro:property name="wheelbase" value="0.40"/>  <!-- 앞/뒤 축 간 거리 (m) -->
+  <xacro:property name="track" value="0.26"/>      <!-- 좌/우 바퀴 간 거리 (m) -->
+  <xacro:property name="wheel_vertical_offset" value="-0.12"/>
+  <!-- 휠 치수 -->
+  <xacro:property name="wheel_length" value="0.045"/>
+  <xacro:property name="wheel_radius" value="0.045"/>
+  <!-- ===== Base frames ===== -->
+  <link name="base_footprint"/>
+  <joint name="base_joint" type="fixed">
     <parent link="base_footprint"/>
     <child link="base_link"/>
-    <origin xyz="0.0 0.0 0.15" rpy="0 0 0"/>
-    </joint>
-    <!-- Base link -->
-    <link name="base_link">
+    <origin xyz="0 0 0.15" rpy="0 0 0"/>
+  </joint>
+  <link name="base_link">
     <inertial>
-      <origin xyz="0 0 -0.05" rpy="0 0 0"/>
+      <origin xyz="0 0 0" rpy="0 0 0"/>
       <mass value="10.0"/>
-      <inertia ixx="0.0203333333" ixy="0" ixz="0"
-               iyy="0.0224166667" iyz="0"
-               izz="0.0260833333"/>
+      <inertia ixx="0.0203333333" ixy="0" ixz="0" iyy="0.0224166667" iyz="0" izz="0.0260833333"/>
     </inertial>
-        <visual>
-            <origin xyz="0 0 -0.15" rpy="0 0 1.57" />
-            <geometry>
-                <mesh filename="package://limo_description/meshes/limo_base.dae" scale="1 1 1"/>
-            </geometry>
-        </visual>
-        <collision>
-            <origin xyz="0 0 0" rpy="0 0 0" />
-          <geometry>
-              <box size="${base_x_size} ${base_y_size} ${base_z_size}"/>
-          </geometry>
-        </collision>
-    </link>
-    <link name="inertial_link">
-        <inertial>
-            <origin xyz="0.0 0.0 0.0" />
-            <mass value="${base_mass}" />
-            <inertia ixx="0.24" ixy="0" ixz="0"
-                     iyy="0.96" iyz="0"
-                     izz="0.96" />
-        </inertial>
-    </link>
-    <joint name="inertial_joint" type="fixed">
-        <origin xyz="0 0 0" rpy="0 0 0" />
-        <parent link="base_link" />
-        <child link="inertial_link" />
-    </joint>
-    <xacro:limo_laser parent_prefix="base_link" frame_prefix="laser">
-        <origin xyz="0.103 0 -0.034" rpy="0 0 0"/>
-    </xacro:limo_laser>
-    <xacro:limo_depth_camera parent_prefix="base_link" frame_prefix="depth_camera">
-        <origin xyz="0.084 0 0.03" rpy="0 0 0"/>
-    </xacro:limo_depth_camera>
-    <xacro:limo_imu parent_prefix="base_link" frame_prefix="imu">
-        <origin xyz="0.0 0 -0.1" rpy="0 0 0"/>
-    </xacro:limo_imu>
-    <xacro:limo_left_steering_hinge parent_prefix="base_link" wheel_prefix="left_steering_hinge">
-        <origin xyz="${wheelbase/2} ${track/2} ${wheel_vertical_offset}" rpy="0 0  0" />
-    </xacro:limo_left_steering_hinge>
-    <xacro:limo_right_steering_hinge parent_prefix="base_link" wheel_prefix="right_steering_hinge">
-        <origin xyz="${wheelbase/2} ${-track/2} ${wheel_vertical_offset}" rpy="${M_PI} 0 0" />
-    </xacro:limo_right_steering_hinge>
-    <link name="rear_left_wheel_link">
-        <inertial>
-            <origin xyz="0 0 0" />
-            <mass value="0.5" />
-            <inertia ixx="0.01055" ixy="0" ixz="0" iyy="0.00075" iyz="0" izz="0.01055" />
-        </inertial>
-        <visual>
-            <origin xyz="0 0 0" rpy="0 0 0" />
-            <geometry>
-                <mesh filename="package://limo_description/meshes/limo_wheel.dae" />
-            </geometry>
-        </visual>
-        <collision>
-            <origin xyz="0 ${wheel_length/2} 0" rpy="1.57 0 0" />
-          <geometry>
-              <cylinder length="${wheel_length}" radius="${wheel_radius}" />
-          </geometry>
-        </collision>
-    </link>
-    <joint name="rear_left_wheel" type="continuous">
-        <parent link="base_link"/>
-        <child link="rear_left_wheel_link"/>
-        <origin xyz="${-wheelbase/2} ${track/2} ${wheel_vertical_offset}" rpy="0 0 0" />
-        <axis xyz="0 1 0"/>
-    </joint>
-    <link name="rear_right_wheel_link">
-        <inertial>
-            <origin xyz="0 0 0" />
-            <mass value="0.5" />
-            <inertia ixx="0.01055" ixy="0" ixz="0" iyy="0.00075" iyz="0" izz="0.01055" />
-        </inertial>
-        <visual>
-            <origin xyz="0 0 0" rpy="0 0 0" />
-            <geometry>
-                <mesh filename="package://limo_description/meshes/limo_wheel.dae" />
-            </geometry>
-        </visual>
-            <collision>
-                <origin xyz="0 ${wheel_length/2} 0" rpy="1.57 0 0" />
-              <geometry>
-                  <cylinder length="${wheel_length}" radius="${wheel_radius}" />
-              </geometry>
-            </collision>
-        </link>
-        <joint name="rear_right_wheel" type="continuous">
-            <parent link="base_link"/>
-            <child link="rear_right_wheel_link"/>
-            <origin xyz="${-wheelbase/2} ${-track/2} ${wheel_vertical_offset}" rpy="${M_PI} 0 0" />
-            <axis xyz="0 -1 0"/>
-        </joint>
+    <visual>
+      <origin xyz="0 0 -0.15" rpy="0 0 1.57"/>
+      <geometry>
+        <mesh filename="package://limo_description/meshes/limo_base.dae" scale="1 1 1"/>
+      </geometry>
+    </visual>
+    <collision>
+      <origin xyz="0 0 0" rpy="0 0 0"/>
+      <geometry>
+        <box size="${base_x_size} ${base_y_size} ${base_z_size}"/>
+      </geometry>
+    </collision>
+  </link>
+  <!-- ===== Front steering (Ackermann): steering hinge + wheel (구동) ===== -->
+  <!-- 왼쪽 앞바퀴: 힌지 링크를 먼저 만들고 그 밑에 휠(구동) 조인트가 매크로 안에서 생성됨 -->
+  <xacro:limo_left_steering_hinge parent_prefix="base_link" wheel_prefix="left_steering_hinge">
+    <origin xyz="${wheelbase/2} ${track/2} ${wheel_vertical_offset}" rpy="0 0 0"/>
+  </xacro:limo_left_steering_hinge>
+  <!-- 오른쪽 앞바퀴: 반대측, 메시 방향 맞추기 위해 rpy의 roll을 PI로 -->
+  <xacro:limo_right_steering_hinge parent_prefix="base_link" wheel_prefix="right_steering_hinge">
+    <origin xyz="${wheelbase/2} ${-track/2} ${wheel_vertical_offset}" rpy="${M_PI} 0 0"/>
+  </xacro:limo_right_steering_hinge>
+  <!-- ===== Rear wheels (구동만, 조향 없음) ===== -->
+  <link name="rear_left_wheel_link">
+    <inertial>
+      <origin xyz="0 0 0"/>
+      <mass value="0.5"/>
+      <inertia ixx="0.01055" ixy="0" ixz="0" iyy="0.00075" iyz="0" izz="0.01055"/>
+    </inertial>
+    <visual>
+      <origin xyz="0 0 0" rpy="0 0 0"/>
+      <geometry>
+        <mesh filename="package://limo_description/meshes/limo_wheel.dae"/>
+      </geometry>
+    </visual>
+    <collision>
+      <origin xyz="0 0 0"/>
+      <geometry>
+        <cylinder length="${wheel_length}" radius="${wheel_radius}"/>
+      </geometry>
+    </collision>
+  </link>
+  <joint name="rear_left_wheel" type="continuous">
+    <parent link="base_link"/>
+    <child link="rear_left_wheel_link"/>
+    <origin xyz="${-wheelbase/2} ${track/2} ${wheel_vertical_offset}" rpy="0 0 0"/>
+    <axis xyz="0 1 0"/>
+  </joint>
+  <link name="rear_right_wheel_link">
+    <inertial>
+      <origin xyz="0 0 0"/>
+      <mass value="0.5"/>
+      <inertia ixx="0.01055" ixy="0" ixz="0" iyy="0.00075" iyz="0" izz="0.01055"/>
+    </inertial>
+    <visual>
+      <origin xyz="0 0 0" rpy="0 0 0"/>
+      <geometry>
+        <mesh filename="package://limo_description/meshes/limo_wheel.dae"/>
+      </geometry>
+    </visual>
+    <collision>
+      <origin xyz="0 0 0"/>
+      <geometry>
+        <cylinder length="${wheel_length}" radius="${wheel_radius}"/>
+      </geometry>
+    </collision>
+  </link>
+  <joint name="rear_right_wheel" type="continuous">
+    <parent link="base_link"/>
+    <child link="rear_right_wheel_link"/>
+    <origin xyz="${-wheelbase/2} ${-track/2} ${wheel_vertical_offset}" rpy="0 0 0"/>
+    <axis xyz="0 -1 0"/>
+  </joint>
+  <!-- ===== Gazebo 플러그인/마찰 세팅: 반드시 모든 변수/조인트 정의 이후에 include ===== -->
+  <!-- 충돌 회피용: 환경 꼬일 때는 아래 주석 한 줄을 풀어 "절대경로 include"로 먼저 테스트 -->
+  <!-- <xacro:include filename="/home/robotu/2lo/limo_ros2/limo_description/urdf/limo_ackerman.gazebo"/> -->
+  <xacro:include filename="$(find limo_description)/urdf/limo_ackerman.gazebo"/>
 </robot>

Commit message: auto commit: 2025-09-18 17:02:38

File: limo_ros2/limo_description/urdf/limo_ackerman.xacro (robot description, xacro)
@@ -3,17 +3,15 @@
   <!-- Args -->
   <xacro:arg name="robot_namespace" default="/limo"/>
-  <!-- Common macros (바퀴/힌지 링크 생성 매크로 포함) -->
+  <!-- Common macros -->
   <xacro:include filename="$(find limo_description)/urdf/limo_xacro.xacro"/>
   <xacro:include filename="$(find limo_description)/urdf/limo_steering_hinge.xacro"/>
-  <!-- ===== Vehicle parameters (변수는 include 전에 선언되어야 함) ===== -->
+  <!-- ===== Vehicle parameters ===== -->
   <xacro:property name="M_PI" value="3.141592653589793"/>
   <xacro:property name="base_x_size" value="0.13"/>
   <xacro:property name="base_y_size" value="0.12"/>
   <xacro:property name="base_z_size" value="0.10"/>
-  <!-- 차체 치수 -->
-  <xacro:property name="wheelbase" value="0.40"/>  <!-- 앞/뒤 축 간 거리 (m) -->
-  <xacro:property name="track" value="0.26"/>      <!-- 좌/우 바퀴 간 거리 (m) -->
+  <xacro:property name="wheelbase" value="0.40"/>
+  <xacro:property name="track" value="0.26"/>
   <xacro:property name="wheel_vertical_offset" value="-0.12"/>
-  <!-- 휠 치수 -->
   <xacro:property name="wheel_length" value="0.045"/>
   <xacro:property name="wheel_radius" value="0.045"/>
@@ -44,14 +42,12 @@
     </collision>
   </link>
-  <!-- ===== Front steering (Ackermann): steering hinge + wheel (구동) ===== -->
-  <!-- 왼쪽 앞바퀴: 힌지 링크를 먼저 만들고 그 밑에 휠(구동) 조인트가 매크로 안에서 생성됨 -->
-  <xacro:limo_left_steering_hinge parent_prefix="base_link" wheel_prefix="left_steering_hinge">
+  <!-- ===== Front steering (Ackermann) ===== -->
+  <xacro:limo_left_steering_hinge parent_prefix="base_link" wheel_prefix="left_steering_joint">
     <origin xyz="${wheelbase/2} ${track/2} ${wheel_vertical_offset}" rpy="0 0 0"/>
   </xacro:limo_left_steering_hinge>
-  <!-- 오른쪽 앞바퀴: 반대측, 메시 방향 맞추기 위해 rpy의 roll을 PI로 -->
-  <xacro:limo_right_steering_hinge parent_prefix="base_link" wheel_prefix="right_steering_hinge">
+  <xacro:limo_right_steering_hinge parent_prefix="base_link" wheel_prefix="right_steering_joint">
     <origin xyz="${wheelbase/2} ${-track/2} ${wheel_vertical_offset}" rpy="${M_PI} 0 0"/>
   </xacro:limo_right_steering_hinge>
-  <!-- ===== Rear wheels (구동만, 조향 없음) ===== -->
+  <!-- ===== Rear wheels ===== -->
   <link name="rear_left_wheel_link">
     <inertial>
@@ -61,5 +57,4 @@
     </inertial>
     <visual>
-      <origin xyz="0 0 0" rpy="0 0 0"/>
       <geometry>
         <mesh filename="package://limo_description/meshes/limo_wheel.dae"/>
@@ -67,5 +62,4 @@
     </visual>
     <collision>
-      <origin xyz="0 0 0"/>
       <geometry>
         <cylinder length="${wheel_length}" radius="${wheel_radius}"/>
@@ -73,5 +67,5 @@
     </collision>
   </link>
-  <joint name="rear_left_wheel" type="continuous">
+  <joint name="rear_left_joint" type="continuous">
     <parent link="base_link"/>
     <child link="rear_left_wheel_link"/>
@@ -86,5 +80,4 @@
     </inertial>
     <visual>
-      <origin xyz="0 0 0" rpy="0 0 0"/>
       <geometry>
         <mesh filename="package://limo_description/meshes/limo_wheel.dae"/>
@@ -92,5 +85,4 @@
     </visual>
     <collision>
-      <origin xyz="0 0 0"/>
       <geometry>
         <cylinder length="${wheel_length}" radius="${wheel_radius}"/>
@@ -98,5 +90,5 @@
     </collision>
   </link>
-  <joint name="rear_right_wheel" type="continuous">
+  <joint name="rear_right_joint" type="continuous">
     <parent link="base_link"/>
     <child link="rear_right_wheel_link"/>
@@ -104,7 +96,5 @@
     <axis xyz="0 -1 0"/>
   </joint>
-  <!-- ===== Gazebo 플러그인/마찰 세팅: 반드시 모든 변수/조인트 정의 이후에 include ===== -->
-  <!-- 충돌 회피용: 환경 꼬일 때는 아래 주석 한 줄을 풀어 "절대경로 include"로 먼저 테스트 -->
-  <!-- <xacro:include filename="/home/robotu/2lo/limo_ros2/limo_description/urdf/limo_ackerman.gazebo"/> -->
+  <!-- Gazebo 플러그인 include -->
   <xacro:include filename="$(find limo_description)/urdf/limo_ackerman.gazebo"/>
 </robot>
